Commit message: Update local copy of URDF and mesh files and add update script
Add script `update_robot_properties.sh` that updates the URDF and mesh
files and update the file using that script.

File: python/pybullet_fingers/robot_properties_fingers/urdf/finger.urdf (robot description, URDF)
Before this commit: robot finger, 7 links, 6 joints
Links:
- link finger_base_link: geometry collision mesh filename=package://robot_properties_fingers/meshes/stl/SIM__BL-Finge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 scale=1 1 1; visual mesh filename=package://robot_properties_fingers/meshes/stl/SIM__BL-Finge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 scale=1 1 1
- link finger_lower_link: geometry collision mesh filename=package://robot_properties_fingers/meshes/stl/SIM_BL_FINGER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 scale=1 1 1; collision mesh filename=package://robot_properties_fingers/meshes/stl/finger_paddin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 scale=1 1 1
- link finger_middle_link: geometry collision mesh filename=package://robot_properties_fingers/meshes/stl/SIM__BL-Finge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 scale=1 1 1; visual mesh filename=package://robot_properties_fingers/meshes/stl/SIM__BL-Finge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 scale=1 1 1
- link finger_upper_holder_link: geometry collision mesh filename=package://robot_properties_fingers/meshes/stl/BL_Finger_Hol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 scale=1 1 1; visual mesh filename=package://robot_properties_fingers/meshes/stl/BL_Finger_Hol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 scale=1 1 1
- link finger_upper_link: geometry collision mesh filename=package://robot_properties_fingers/meshes/stl/SIM__BL-Finge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 scale=1 1 1; visual mesh filename=package://robot_properties_fingers/meshes/stl/SIM__BL-Finge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 scale=1 1 1

File: python/pybullet_fingers/robot_properties_fingers/urdf/finger_with_stage.urdf (robot description, URDF)
Before this commit: robot finger_with_stage, 8 links, 7 joints
Links:
- link finger_base_link: geometry collision mesh filename=package://robot_properties_fingers/meshes/stl/SIM__BL-Finge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 scale=1 1 1; visual mesh filename=package://robot_properties_fingers/meshes/stl/SIM__BL-Finge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 scale=1 1 1
- link finger_lower_link: geometry collision mesh filename=package://robot_properties_fingers/meshes/stl/SIM_BL_FINGER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 scale=1 1 1; collision mesh filename=package://robot_properties_fingers/meshes/stl/finger_paddin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 scale=1 1 1
- link finger_middle_link: geometry collision mesh filename=package://robot_properties_fingers/meshes/stl/SIM__BL-Finge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 scale=1 1 1; visual mesh filename=package://robot_properties_fingers/meshes/stl/SIM__BL-Finge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 scale=1 1 1
- link finger_upper_holder_link: geometry collision mesh filename=package://robot_properties_fingers/meshes/stl/BL_Finger_Hol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 scale=1 1 1; visual mesh filename=package://robot_properties_fingers/meshes/stl/BL_Finger_Hol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 scale=1 1 1
- link finger_upper_link: geometry collision mesh filename=package://robot_properties_fingers/meshes/stl/SIM__BL-Finge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 scale=1 1 1; visual mesh filename=package://robot_properties_fingers/meshes/stl/SIM__BL-Finge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 scale=1 1 1
- link stage_link: geometry collision mesh filename=package://robot_properties_fingers/meshes/stl/Stage_simplif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 scale=1 1 1; visual mesh filename=package://robot_properties_fingers/meshes/stl/Stage_simplif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 scale=1 1 1

File: python/pybullet_fingers/robot_properties_fingers/urdf/stage.urdf (robot description, URDF)
Before this commit: robot stage, 1 links, 0 joints
Links:
- link stage_link: geometry collision mesh filename=package://robot_properties_fingers/meshes/stl/Stage_simplif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 scale=1 1 1; visual mesh filename=package://robot_properties_fingers/meshes/stl/Stage_simplif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 scale=1 1 1

File: python/pybullet_fingers/robot_properties_fingers/urdf/trifinger.urdf (robot description, URDF)
Before this commit: robot finger_with_stage, 17 links, 16 joints
Links:
- link finger_base_link_0: geometry collision mesh filename=package://robot_properties_fingers/meshes/stl/SIM__BL-Finge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 scale=1 1 1; visual mesh filename=package://robot_properties_fingers/meshes/stl/SIM__BL-Finge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 scale=1 1 1
- link finger_base_link_120: geometry collision mesh filename=package://robot_properties_fingers/meshes/stl/SIM__BL-Finge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 scale=1 1 1; visual mesh filename=package://robot_properties_fingers/meshes/stl/SIM__BL-Finge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 scale=1 1 1
- link finger_base_link_240: geometry collision mesh filename=package://robot_properties_fingers/meshes/stl/SIM__BL-Finge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 scale=1 1 1; visual mesh filename=package://robot_properties_fingers/meshes/stl/SIM__BL-Finge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 scale=1 1 1
- link finger_lower_link_0: geometry collision mesh filename=package://robot_properties_fingers/meshes/stl/SIM_BL_FINGER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 scale=1 1 1; visual mesh filename=package://robot_properties_fingers/meshes/stl/SIM_BL_FINGER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 scale=1 1 1
- link finger_lower_link_120: geometry collision mesh filename=package://robot_properties_fingers/meshes/stl/SIM_BL_FINGER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 scale=1 1 1; visual mesh filename=package://robot_properties_fingers/meshes/stl/SIM_BL_FINGER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 scale=1 1 1
- link finger_lower_link_240: geometry collision mesh filename=package://robot_properties_fingers/meshes/stl/SIM_BL_FINGER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 scale=1 1 1; visual mesh filename=package://robot_properties_fingers/meshes/stl/SIM_BL_FINGER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 scale=1 1 1
- link finger_middle_link_0: geometry collision mesh filename=package://robot_properties_fingers/meshes/stl/SIM__BL-Finge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 scale=1 1 1; visual mesh filename=package://robot_properties_fingers/meshes/stl/SIM__BL-Finge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 scale=1 1 1
- link finger_middle_link_120: geometry collision mesh filename=package://robot_properties_fingers/meshes/stl/SIM__BL-Finge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 scale=1 1 1; visual mesh filename=package://robot_properties_fingers/meshes/stl/SIM__BL-Finge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 scale=1 1 1
- link finger_middle_link_240: geometry collision mesh filename=package://robot_properties_fingers/meshes/stl/SIM__BL-Finge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 scale=1 1 1; visual mesh filename=package://robot_properties_fingers/meshes/stl/SIM__BL-Finge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 scale=1 1 1
- link finger_upper_link_0: geometry collision mesh filename=package://robot_properties_fingers/meshes/stl/SIM__BL-Finge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 scale=1 1 1; visual mesh filename=package://robot_properties_fingers/meshes/stl/SIM__BL-Finge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 scale=1 1 1
- link finger_upper_link_120: geometry collision mesh filename=package://robot_properties_fingers/meshes/stl/SIM__BL-Finge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 scale=1 1 1; visual mesh filename=package://robot_properties_fingers/meshes/stl/SIM__BL-Finge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 scale=1 1 1
- link finger_upper_link_240: geometry collision mesh filename=package://robot_properties_fingers/meshes/stl/SIM__BL-Finge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 scale=1 1 1; visual mesh filename=package://robot_properties_fingers/meshes/stl/SIM__BL-Finge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 scale=1 1 1

File: python/pybullet_fingers/robot_properties_fingers/urdf/trifinger_with_stage.urdf (robot description, URDF)
Before this commit: robot finger_with_stage, 18 links, 17 joints
Links:
- link finger_base_link_0: geometry collision mesh filename=package://robot_properties_fingers/meshes/stl/SIM__BL-Finge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 scale=1 1 1; visual mesh filename=package://robot_properties_fingers/meshes/stl/SIM__BL-Finge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 scale=1 1 1
- link finger_base_link_120: geometry collision mesh filename=package://robot_properties_fingers/meshes/stl/SIM__BL-Finge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 scale=1 1 1; visual mesh filename=package://robot_properties_fingers/meshes/stl/SIM__BL-Finge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 scale=1 1 1
- link finger_base_link_240: geometry collision mesh filename=package://robot_properties_fingers/meshes/stl/SIM__BL-Finge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 scale=1 1 1; visual mesh filename=package://robot_properties_fingers/meshes/stl/SIM__BL-Finge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 scale=1 1 1
- link finger_lower_link_0: geometry collision mesh filename=package://robot_properties_fingers/meshes/stl/SIM_BL_FINGER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 scale=1 1 1; visual mesh filename=package://robot_properties_fingers/meshes/stl/SIM_BL_FINGER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 scale=1 1 1
- link finger_lower_link_120: geometry collision mesh filename=package://robot_properties_fingers/meshes/stl/SIM_BL_FINGER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 scale=1 1 1; visual mesh filename=package://robot_properties_fingers/meshes/stl/SIM_BL_FINGER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 scale=1 1 1
- link finger_lower_link_240: geometry collision mesh filename=package://robot_properties_fingers/meshes/stl/SIM_BL_FINGER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 scale=1 1 1; visual mesh filename=package://robot_properties_fingers/meshes/stl/SIM_BL_FINGER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 scale=1 1 1
- link finger_middle_link_0: geometry collision mesh filename=package://robot_properties_fingers/meshes/stl/SIM__BL-Finge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 scale=1 1 1; visual mesh filename=package://robot_properties_fingers/meshes/stl/SIM__BL-Finge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 scale=1 1 1
- link finger_middle_link_120: geometry collision mesh filename=package://robot_properties_fingers/meshes/stl/SIM__BL-Finge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 scale=1 1 1; visual mesh filename=package://robot_properties_fingers/meshes/stl/SIM__BL-Finge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 scale=1 1 1
- link finger_middle_link_240: geometry collision mesh filename=package://robot_properties_fingers/meshes/stl/SIM__BL-Finge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 scale=1 1 1; visual mesh filename=package://robot_properties_fingers/meshes/stl/SIM__BL-Finge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 scale=1 1 1
- link finger_upper_link_0: geometry collision mesh filename=package://robot_properties_fingers/meshes/stl/SIM__BL-Finge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 scale=1 1 1; visual mesh filename=package://robot_properties_fingers/meshes/stl/SIM__BL-Finge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 scale=1 1 1
- link finger_upper_link_120: geometry collision mesh filename=package://robot_properties_fingers/meshes/stl/SIM__BL-Finge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 scale=1 1 1; visual mesh filename=package://robot_properties_fingers/meshes/stl/SIM__BL-Finge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 scale=1 1 1
- link finger_upper_link_240: geometry collision mesh filename=package://robot_properties_fingers/meshes/stl/SIM__BL-Finge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 scale=1 1 1; visual mesh filename=package://robot_properties_fingers/meshes/stl/SIM__BL-Finge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 scale=1 1 1
- link stage_link: geometry collision mesh filename=package://robot_properties_fingers/meshes/stl/BL-M_Table_AS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 scale=1 1 1; visual mesh filename=package://robot_properties_fingers/meshes/stl/BL-M_Table_AS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 scale=1 1 1

Commit message: Update copy of URDF and mesh files
This now also includes the FingerEdu files.

File: python/pybullet_fingers/robot_properties_fingers/urdf/finger.urdf (robot description, URDF)
Before this commit: robot finger, 7 links, 6 joints
Joints:
- joint finger_middle_to_lower_joint: limit lower=-3.00196631343 upper=-0.0349065850399 effort=1000 velocity=1000 -> lower=-3.00196631343 upper=3.00196631343 effort=1000 velocity=1000

File: python/pybullet_fingers/robot_properties_fingers/urdf/finger_with_stage.urdf (robot description, URDF)
Before this commit: robot finger_with_stage, 8 links, 7 joints
Joints:
- joint finger_middle_to_lower_joint: limit lower=-3.00196631343 upper=-0.0349065850399 effort=1000 velocity=1000 -> lower=-3.00196631343 upper=3.00196631343 effort=1000 velocity=1000

File: python/pybullet_fingers/robot_properties_fingers/urdf/trifinger.urdf (robot description, URDF)
Before this commit: robot finger_with_stage, 17 links, 16 joints
Joints:
- joint finger_middle_to_lower_joint_0: limit lower=-3.00196631343 upper=-0.0349065850399 effort=1000 velocity=1000 -> lower=-3.00196631343 upper=3.00196631343 effort=1000 velocity=1000
- joint finger_middle_to_lower_joint_120: limit lower=-3.00196631343 upper=-0.0349065850399 effort=1000 velocity=1000 -> lower=-3.00196631343 upper=3.00196631343 effort=1000 velocity=1000
- joint finger_middle_to_lower_joint_240: limit lower=-3.00196631343 upper=-0.0349065850399 effort=1000 velocity=1000 -> lower=-3.00196631343 upper=3.00196631343 effort=1000 velocity=1000

File: python/pybullet_fingers/robot_properties_fingers/urdf/trifinger_with_stage.urdf (robot description, URDF)
Before this commit: robot finger_with_stage, 18 links, 17 joints
Links:
- removed link stage_link
- added link boundary_link, mass 2; collision mesh filename=package://robot_properties_fingers/meshes/stl/high_table_bo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 scale=1 1 1; visual mesh filename=package://robot_properties_fingers/meshes/stl/high_table_bo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 scale=1 1 1
- added link table_link, mass 2; collision mesh filename=package://robot_properties_fingers/meshes/stl/trifinger_tab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 scale=1 1 1; visual mesh filename=package://robot_properties_fingers/meshes/stl/trifinger_tab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 scale=1 1 1
Joints:
- removed joint base_to_stage
- added joint base_to_table: type fixed, parent base_link, child table_link, origin xyz=0 0 0
- added joint table_to_boundary: type fixed, parent table_link, child boundary_link, origin xyz=0 0 0
- joint finger_middle_to_lower_joint_0: limit lower=-3.00196631343 upper=-0.0349065850399 effort=1000 velocity=1000 -> lower=-3.00196631343 upper=3.00196631343 effort=1000 velocity=1000
- joint finger_middle_to_lower_joint_120: limit lower=-3.00196631343 upper=-0.0349065850399 effort=1000 velocity=1000 -> lower=-3.00196631343 upper=3.00196631343 effort=1000 velocity=1000
- joint finger_middle_to_lower_joint_240: limit lower=-3.00196631343 upper=-0.0349065850399 effort=1000 velocity=1000 -> lower=-3.00196631343 upper=3.00196631343 effort=1000 velocity=1000
