Commit message: Update URDF models
Using the models of robot_properties_fingers revision bff387ee.
Most relevant change: Add the TriFingerPro model.

File: python/pybullet_fingers/robot_properties_fingers/urdf/pro/trifingerpro.urdf (robot description, URDF)
Before this commit: robot finger_with_stage, 17 links, 16 joints
Links:
- link finger_base_link_0: geometry collision mesh filename=package://robot_properties_fingers/meshes/stl/pro/SIM__BL-F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 scale=1.0 1.0 1.0; visual mesh filename=package://robot_properties_fingers/meshes/stl/pro/SIM__BL-F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 scale=1.0 1.0 1.0
- link finger_base_link_120: geometry collision mesh filename=package://robot_properties_fingers/meshes/stl/pro/SIM__BL-F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 scale=1.0 1.0 1.0; visual mesh filename=package://robot_properties_fingers/meshes/stl/pro/SIM__BL-F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 scale=1.0 1.0 1.0
- link finger_base_link_240: geometry collision mesh filename=package://robot_properties_fingers/meshes/stl/pro/SIM__BL-F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 scale=1.0 1.0 1.0; visual mesh filename=package://robot_properties_fingers/meshes/stl/pro/SIM__BL-F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 scale=1.0 1.0 1.0
- link finger_lower_link_0: geometry collision mesh filename=package://robot_properties_fingers/meshes/stl/pro/SIM__BL-F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 scale=1.0 1.0 1.0; visual mesh filename=package://robot_properties_fingers/meshes/stl/pro/SIM__BL-F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 scale=1.0 1.0 1.0
- link finger_lower_link_120: geometry collision mesh filename=package://robot_properties_fingers/meshes/stl/pro/SIM__BL-F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 scale=1.0 1.0 1.0; visual mesh filename=package://robot_properties_fingers/meshes/stl/pro/SIM__BL-F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 scale=1.0 1.0 1.0
- link finger_lower_link_240: geometry collision mesh filename=package://robot_properties_fingers/meshes/stl/pro/SIM__BL-F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 scale=1.0 1.0 1.0; visual mesh filename=package://robot_properties_fingers/meshes/stl/pro/SIM__BL-F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 scale=1.0 1.0 1.0
- link finger_middle_link_0: geometry collision mesh filename=package://robot_properties_fingers/meshes/stl/pro/SIM__BL-F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 scale=1.0 1.0 1.0; visual mesh filename=package://robot_properties_fingers/meshes/stl/pro/SIM__BL-F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 scale=1.0 1.0 1.0
- link finger_middle_link_120: geometry collision mesh filename=package://robot_properties_fingers/meshes/stl/pro/SIM__BL-F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 scale=1.0 1.0 1.0; visual mesh filename=package://robot_properties_fingers/meshes/stl/pro/SIM__BL-F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 scale=1.0 1.0 1.0
- link finger_middle_link_240: geometry collision mesh filename=package://robot_properties_fingers/meshes/stl/pro/SIM__BL-F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 scale=1.0 1.0 1.0; visual mesh filename=package://robot_properties_fingers/meshes/stl/pro/SIM__BL-F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 scale=1.0 1.0 1.0
- link finger_upper_link_0: geometry collision mesh filename=package://robot_properties_fingers/meshes/stl/pro/SIM__BL-F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 scale=1.0 1.0 1.0; visual mesh filename=package://robot_properties_fingers/meshes/stl/pro/SIM__BL-F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 scale=1.0 1.0 1.0
- link finger_upper_link_120: geometry collision mesh filename=package://robot_properties_fingers/meshes/stl/pro/SIM__BL-F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 scale=1.0 1.0 1.0; visual mesh filename=package://robot_properties_fingers/meshes/stl/pro/SIM__BL-F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 scale=1.0 1.0 1.0
- link finger_upper_link_240: geometry collision mesh filename=package://robot_properties_fingers/meshes/stl/pro/SIM__BL-F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 scale=1.0 1.0 1.0; visual mesh filename=package://robot_properties_fingers/meshes/stl/pro/SIM__BL-F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 scale=1.0 1.0 1.0
- link upper_holder_link: geometry visual mesh filename=package://robot_properties_fingers/meshes/stl/pro/SIM__BL-F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 scale=1.0 1.0 1.0
Joints:
- joint base_to_upper_holder_joint: origin xyz=0 0 0.34 -> xyz=0 0 0.29
- joint finger_base_to_upper_joint_0: limit lower=-1.57079632679 upper=1.57079632679 effort=1000 velocity=1000 -> lower=-0.9 upper=1.4 effort=1000 velocity=1000
- joint finger_base_to_upper_joint_120: limit lower=-1.57079632679 upper=1.57079632679 effort=1000 velocity=1000 -> lower=-0.9 upper=1.4 effort=1000 velocity=1000
- joint finger_base_to_upper_joint_240: limit lower=-1.57079632679 upper=1.57079632679 effort=1000 velocity=1000 -> lower=-0.9 upper=1.4 effort=1000 velocity=1000
- joint finger_lower_to_tip_joint_0: origin xyz=0 0 -0.16 -> xyz=0.0185 0 -0.16
- joint finger_lower_to_tip_joint_120: origin xyz=0 0 -0.16 -> xyz=0.0185 0 -0.16
- joint finger_lower_to_tip_joint_240: origin xyz=0 0 -0.16 -> xyz=0.0185 0 -0.16
- joint finger_middle_to_lower_joint_0: limit lower=-3.00196631343 upper=3.00196631343 effort=1000 velocity=1000 -> lower=-2.7 upper=2.7 effort=1000 velocity=1000; origin xyz=0 0 -0.16 rpy=0 0 0 -> xyz=0.04922 0 -0.16 rpy=0 0 0
- joint finger_middle_to_lower_joint_120: limit lower=-3.00196631343 upper=3.00196631343 effort=1000 velocity=1000 -> lower=-2.7 upper=2.7 effort=1000 velocity=1000; origin xyz=0 0 -0.16 rpy=0 0 0 -> xyz=0.04922 0 -0.16 rpy=0 0 0
- joint finger_middle_to_lower_joint_240: limit lower=-3.00196631343 upper=3.00196631343 effort=1000 velocity=1000 -> lower=-2.7 upper=2.7 effort=1000 velocity=1000; origin xyz=0 0 -0.16 rpy=0 0 0 -> xyz=0.04922 0 -0.16 rpy=0 0 0
- joint finger_upper_to_middle_joint_0: axis -1 0 0 -> 1 0 0; limit lower=-1.3526301703 upper=4.49422282389 effort=1000 velocity=1000 -> lower=-1.57 upper=1.57 effort=1000 velocity=1000; origin xyz=0 0 0 rpy=0 0 0 -> xyz=0.01685 0.0505 0 rpy=0 0 0
- joint finger_upper_to_middle_joint_120: axis -1 0 0 -> 1 0 0; limit lower=-1.3526301703 upper=4.49422282389 effort=1000 velocity=1000 -> lower=-1.57 upper=1.57 effort=1000 velocity=1000; origin xyz=0 0 0 rpy=0 0 0 -> xyz=0.01685 0.0505 0 rpy=0 0 0
- joint finger_upper_to_middle_joint_240: axis -1 0 0 -> 1 0 0; limit lower=-1.3526301703 upper=4.49422282389 effort=1000 velocity=1000 -> lower=-1.57 upper=1.57 effort=1000 velocity=1000; origin xyz=0 0 0 rpy=0 0 0 -> xyz=0.01685 0.0505 0 rpy=0 0 0
- joint holder_to_finger_0: origin xyz=0.0 0.04 0 rpy=0 0 0 -> xyz=0 0 0 rpy=0 0 0.0
- joint holder_to_finger_120: origin xyz=0.0346410161514 -0.02 0 rpy=0 0 -2.09439510239 -> xyz=0 0 0 rpy=0 0 -2.09439510239
- joint holder_to_finger_240: origin xyz=-0.0346410161514 -0.02 0 rpy=0 0 -4.18879020479 -> xyz=0 0 0 rpy=0 0 -4.18879020479

File: python/pybullet_fingers/robot_properties_fingers/urdf/pro/trifingerpro_with_stage.urdf (robot description, URDF)
Before this commit: robot finger_with_stage, 17 links, 16 joints
Links:
- added link boundary_link, mass 2; collision mesh filename=package://robot_properties_fingers/meshes/stl/high_table_bo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 scale=1 1 1; visual mesh filename=package://robot_properties_fingers/meshes/stl/high_table_bo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 scale=1 1 1
- added link table_link, mass 2; collision mesh filename=package://robot_properties_fingers/meshes/stl/trifinger_tab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 scale=1 1 1; visual mesh filename=package://robot_properties_fingers/meshes/stl/trifinger_tab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 scale=1 1 1
- link finger_base_link_0: geometry collision mesh filename=package://robot_properties_fingers/meshes/stl/pro/SIM__BL-F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 scale=1.0 1.0 1.0; visual mesh filename=package://robot_properties_fingers/meshes/stl/pro/SIM__BL-F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 scale=1.0 1.0 1.0
- link finger_base_link_120: geometry collision mesh filename=package://robot_properties_fingers/meshes/stl/pro/SIM__BL-F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 scale=1.0 1.0 1.0; visual mesh filename=package://robot_properties_fingers/meshes/stl/pro/SIM__BL-F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 scale=1.0 1.0 1.0
- link finger_base_link_240: geometry collision mesh filename=package://robot_properties_fingers/meshes/stl/pro/SIM__BL-F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 scale=1.0 1.0 1.0; visual mesh filename=package://robot_properties_fingers/meshes/stl/pro/SIM__BL-F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 scale=1.0 1.0 1.0
- link finger_lower_link_0: geometry collision mesh filename=package://robot_properties_fingers/meshes/stl/pro/SIM__BL-F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 scale=1.0 1.0 1.0; visual mesh filename=package://robot_properties_fingers/meshes/stl/pro/SIM__BL-F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 scale=1.0 1.0 1.0
- link finger_lower_link_120: geometry collision mesh filename=package://robot_properties_fingers/meshes/stl/pro/SIM__BL-F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 scale=1.0 1.0 1.0; visual mesh filename=package://robot_properties_fingers/meshes/stl/pro/SIM__BL-F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 scale=1.0 1.0 1.0
- link finger_lower_link_240: geometry collision mesh filename=package://robot_properties_fingers/meshes/stl/pro/SIM__BL-F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 scale=1.0 1.0 1.0; visual mesh filename=package://robot_properties_fingers/meshes/stl/pro/SIM__BL-F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 scale=1.0 1.0 1.0
- link finger_middle_link_0: geometry collision mesh filename=package://robot_properties_fingers/meshes/stl/pro/SIM__BL-F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 scale=1.0 1.0 1.0; visual mesh filename=package://robot_properties_fingers/meshes/stl/pro/SIM__BL-F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 scale=1.0 1.0 1.0
- link finger_middle_link_120: geometry collision mesh filename=package://robot_properties_fingers/meshes/stl/pro/SIM__BL-F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 scale=1.0 1.0 1.0; visual mesh filename=package://robot_properties_fingers/meshes/stl/pro/SIM__BL-F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 scale=1.0 1.0 1.0
- link finger_middle_link_240: geometry collision mesh filename=package://robot_properties_fingers/meshes/stl/pro/SIM__BL-F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 scale=1.0 1.0 1.0; visual mesh filename=package://robot_properties_fingers/meshes/stl/pro/SIM__BL-F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 scale=1.0 1.0 1.0
- link finger_upper_link_0: geometry collision mesh filename=package://robot_properties_fingers/meshes/stl/pro/SIM__BL-F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 scale=1.0 1.0 1.0; visual mesh filename=package://robot_properties_fingers/meshes/stl/pro/SIM__BL-F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 scale=1.0 1.0 1.0
- link finger_upper_link_120: geometry collision mesh filename=package://robot_properties_fingers/meshes/stl/pro/SIM__BL-F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 scale=1.0 1.0 1.0; visual mesh filename=package://robot_properties_fingers/meshes/stl/pro/SIM__BL-F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 scale=1.0 1.0 1.0
- link finger_upper_link_240: geometry collision mesh filename=package://robot_properties_fingers/meshes/stl/pro/SIM__BL-F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 scale=1.0 1.0 1.0; visual mesh filename=package://robot_properties_fingers/meshes/stl/pro/SIM__BL-F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 scale=1.0 1.0 1.0
- link upper_holder_link: geometry visual mesh filename=package://robot_properties_fingers/meshes/stl/pro/SIM__BL-F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 scale=1.0 1.0 1.0
Joints:
- added joint base_to_table: type fixed, parent base_link, child table_link, origin xyz=0 0 0
- added joint table_to_boundary: type fixed, parent table_link, child boundary_link, origin xyz=0 0 0
- joint base_to_upper_holder_joint: origin xyz=0 0 0.34 -> xyz=0 0 0.29
- joint finger_base_to_upper_joint_0: limit lower=-1.57079632679 upper=1.57079632679 effort=1000 velocity=1000 -> lower=-0.9 upper=1.4 effort=1000 velocity=1000
- joint finger_base_to_upper_joint_120: limit lower=-1.57079632679 upper=1.57079632679 effort=1000 velocity=1000 -> lower=-0.9 upper=1.4 effort=1000 velocity=1000
- joint finger_base_to_upper_joint_240: limit lower=-1.57079632679 upper=1.57079632679 effort=1000 velocity=1000 -> lower=-0.9 upper=1.4 effort=1000 velocity=1000
- joint finger_lower_to_tip_joint_0: origin xyz=0 0 -0.16 -> xyz=0.0185 0 -0.16
- joint finger_lower_to_tip_joint_120: origin xyz=0 0 -0.16 -> xyz=0.0185 0 -0.16
- joint finger_lower_to_tip_joint_240: origin xyz=0 0 -0.16 -> xyz=0.0185 0 -0.16
- joint finger_middle_to_lower_joint_0: limit lower=-3.00196631343 upper=3.00196631343 effort=1000 velocity=1000 -> lower=-2.7 upper=2.7 effort=1000 velocity=1000; origin xyz=0 0 -0.16 rpy=0 0 0 -> xyz=0.04922 0 -0.16 rpy=0 0 0
- joint finger_middle_to_lower_joint_120: limit lower=-3.00196631343 upper=3.00196631343 effort=1000 velocity=1000 -> lower=-2.7 upper=2.7 effort=1000 velocity=1000; origin xyz=0 0 -0.16 rpy=0 0 0 -> xyz=0.04922 0 -0.16 rpy=0 0 0
- joint finger_middle_to_lower_joint_240: limit lower=-3.00196631343 upper=3.00196631343 effort=1000 velocity=1000 -> lower=-2.7 upper=2.7 effort=1000 velocity=1000; origin xyz=0 0 -0.16 rpy=0 0 0 -> xyz=0.04922 0 -0.16 rpy=0 0 0
- joint finger_upper_to_middle_joint_0: axis -1 0 0 -> 1 0 0; limit lower=-1.3526301703 upper=4.49422282389 effort=1000 velocity=1000 -> lower=-1.57 upper=1.57 effort=1000 velocity=1000; origin xyz=0 0 0 rpy=0 0 0 -> xyz=0.01685 0.0505 0 rpy=0 0 0
- joint finger_upper_to_middle_joint_120: axis -1 0 0 -> 1 0 0; limit lower=-1.3526301703 upper=4.49422282389 effort=1000 velocity=1000 -> lower=-1.57 upper=1.57 effort=1000 velocity=1000; origin xyz=0 0 0 rpy=0 0 0 -> xyz=0.01685 0.0505 0 rpy=0 0 0
- joint finger_upper_to_middle_joint_240: axis -1 0 0 -> 1 0 0; limit lower=-1.3526301703 upper=4.49422282389 effort=1000 velocity=1000 -> lower=-1.57 upper=1.57 effort=1000 velocity=1000; origin xyz=0 0 0 rpy=0 0 0 -> xyz=0.01685 0.0505 0 rpy=0 0 0
- joint holder_to_finger_0: origin xyz=0.0 0.04 0 rpy=0 0 0 -> xyz=0 0 0 rpy=0 0 0.0
- joint holder_to_finger_120: origin xyz=0.0346410161514 -0.02 0 rpy=0 0 -2.09439510239 -> xyz=0 0 0 rpy=0 0 -2.09439510239
- joint holder_to_finger_240: origin xyz=-0.0346410161514 -0.02 0 rpy=0 0 -4.18879020479 -> xyz=0 0 0 rpy=0 0 -4.18879020479

File: python/pybullet_fingers/robot_properties_fingers/urdf/trifinger_with_stage.urdf (robot description, URDF)
Before this commit: robot trifinger_with_stage, 19 links, 18 joints
Links:
- link upper_holder_link: mass None -> 1
