Commit message: Update URDF models
Update to robot_properties_fingers revision 94c1fb93

File: python/pybullet_fingers/robot_properties_fingers/urdf/edu/trifingeredu.urdf (robot description, URDF)
Before this commit: robot trifingeredu, 17 links, 16 joints
Links:
- link trifinger_base_link: mass None -> 1

File: python/pybullet_fingers/robot_properties_fingers/urdf/edu/trifingeredu_with_stage.urdf (robot description, URDF)
Before this commit: robot trifingeredu_with_stage, 19 links, 18 joints
Links:
- link trifinger_base_link: mass None -> 1
