Commit message: fix cube_v2 collision shape and inertial

File: python/trifinger_simulation/data/cube_v2/cube_v2.urdf (robot description, URDF)
Before this commit: robot cube_v2, 1 links, 0 joints
Links:
- link cube: mass 1.094 -> 0.094; geometry collision mesh filename=cube_v2.obj; visual mesh filename=cube_v2.obj
