Commit message: Update local URDF
Based on robot_properties_fingers rev. 3301dffa

File: python/trifinger_simulation/robot_properties_fingers/urdf/pro/fingerpro.urdf (robot description, URDF)
Before this commit: robot fingerpro, 6 links, 5 joints
Links:
- link finger_tip_link: mass 0.02 -> 0
Joints:
- joint finger_lower_to_tip_joint: origin xyz=0.0185 0 -0.16 -> xyz=0.0185 0 -0.1626
- joint finger_middle_to_lower_joint: limit lower=-2.7 upper=2.7 effort=1000 velocity=1000 -> lower=-2.7 upper=0.0 effort=1000 velocity=1000

File: python/trifinger_simulation/robot_properties_fingers/urdf/pro/trifingerpro.urdf (robot description, URDF)
Before this commit: robot trifingerpro, 17 links, 16 joints
Links:
- link finger_tip_link_0: mass 0.02 -> 0
- link finger_tip_link_120: mass 0.02 -> 0
- link finger_tip_link_240: mass 0.02 -> 0
Joints:
- joint finger_lower_to_tip_joint_0: origin xyz=0.0185 0 -0.16 -> xyz=0.0185 0 -0.1626
- joint finger_lower_to_tip_joint_120: origin xyz=0.0185 0 -0.16 -> xyz=0.0185 0 -0.1626
- joint finger_lower_to_tip_joint_240: origin xyz=0.0185 0 -0.16 -> xyz=0.0185 0 -0.1626
- joint finger_middle_to_lower_joint_0: limit lower=-2.7 upper=2.7 effort=1000 velocity=1000 -> lower=-2.7 upper=0.0 effort=1000 velocity=1000
- joint finger_middle_to_lower_joint_120: limit lower=-2.7 upper=2.7 effort=1000 velocity=1000 -> lower=-2.7 upper=0.0 effort=1000 velocity=1000
- joint finger_middle_to_lower_joint_240: limit lower=-2.7 upper=2.7 effort=1000 velocity=1000 -> lower=-2.7 upper=0.0 effort=1000 velocity=1000

File: python/trifinger_simulation/robot_properties_fingers/urdf/pro/trifingerpro_with_stage.urdf (robot description, URDF)
Before this commit: robot trifingerpro_with_stage, 19 links, 18 joints
Links:
- link finger_tip_link_0: mass 0.02 -> 0
- link finger_tip_link_120: mass 0.02 -> 0
- link finger_tip_link_240: mass 0.02 -> 0
Joints:
- joint finger_lower_to_tip_joint_0: origin xyz=0.0185 0 -0.16 -> xyz=0.0185 0 -0.1626
- joint finger_lower_to_tip_joint_120: origin xyz=0.0185 0 -0.16 -> xyz=0.0185 0 -0.1626
- joint finger_lower_to_tip_joint_240: origin xyz=0.0185 0 -0.16 -> xyz=0.0185 0 -0.1626
- joint finger_middle_to_lower_joint_0: limit lower=-2.7 upper=2.7 effort=1000 velocity=1000 -> lower=-2.7 upper=0.0 effort=1000 velocity=1000
- joint finger_middle_to_lower_joint_120: limit lower=-2.7 upper=2.7 effort=1000 velocity=1000 -> lower=-2.7 upper=0.0 effort=1000 velocity=1000
- joint finger_middle_to_lower_joint_240: limit lower=-2.7 upper=2.7 effort=1000 velocity=1000 -> lower=-2.7 upper=0.0 effort=1000 velocity=1000

Commit message: Update robot model to state of robot_properties_fingers@051a702

File: python/trifinger_simulation/robot_properties_fingers/urdf/pro/fingerpro.urdf (robot description, URDF)
Before this commit: robot fingerpro, 6 links, 5 joints
Links:
- link finger_lower_link: mass 0.01 -> 0.021
- link finger_middle_link: mass 0.2 -> 0.25
- link finger_tip_link: mass 0 -> 0.031; geometry collision mesh filename=package://robot_properties_fingers/meshes/stl/pro/SIM__BL-F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 scale=1.0 1.0 1.0; visual mesh filename=package://robot_properties_fingers/meshes/stl/pro/SIM__BL-F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 scale=1.0 1.0 1.0
- link finger_upper_link: mass 0.2 -> 0.26

File: python/trifinger_simulation/robot_properties_fingers/urdf/pro/trifingerpro.urdf (robot description, URDF)
Before this commit: robot trifingerpro, 17 links, 16 joints
Links:
- link finger_lower_link_0: mass 0.01 -> 0.021
- link finger_lower_link_120: mass 0.01 -> 0.021
- link finger_lower_link_240: mass 0.01 -> 0.021
- link finger_middle_link_0: mass 0.2 -> 0.25
- link finger_middle_link_120: mass 0.2 -> 0.25
- link finger_middle_link_240: mass 0.2 -> 0.25
- link finger_tip_link_0: mass 0 -> 0.031; geometry collision mesh filename=package://robot_properties_fingers/meshes/stl/pro/SIM__BL-F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 scale=1.0 1.0 1.0; visual mesh filename=package://robot_properties_fingers/meshes/stl/pro/SIM__BL-F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 scale=1.0 1.0 1.0
- link finger_tip_link_120: mass 0 -> 0.031; geometry collision mesh filename=package://robot_properties_fingers/meshes/stl/pro/SIM__BL-F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 scale=1.0 1.0 1.0; visual mesh filename=package://robot_properties_fingers/meshes/stl/pro/SIM__BL-F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 scale=1.0 1.0 1.0
- link finger_tip_link_240: mass 0 -> 0.031; geometry collision mesh filename=package://robot_properties_fingers/meshes/stl/pro/SIM__BL-F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 scale=1.0 1.0 1.0; visual mesh filename=package://robot_properties_fingers/meshes/stl/pro/SIM__BL-F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 scale=1.0 1.0 1.0
- link finger_upper_link_0: mass 0.2 -> 0.26
- link finger_upper_link_120: mass 0.2 -> 0.26
- link finger_upper_link_240: mass 0.2 -> 0.26

File: python/trifinger_simulation/robot_properties_fingers/urdf/pro/trifingerpro_with_stage.urdf (robot description, URDF)
Before this commit: robot trifingerpro_with_stage, 19 links, 18 joints
Links:
- link finger_lower_link_0: mass 0.01 -> 0.021
- link finger_lower_link_120: mass 0.01 -> 0.021
- link finger_lower_link_240: mass 0.01 -> 0.021
- link finger_middle_link_0: mass 0.2 -> 0.25
- link finger_middle_link_120: mass 0.2 -> 0.25
- link finger_middle_link_240: mass 0.2 -> 0.25
- link finger_tip_link_0: mass 0 -> 0.031; geometry collision mesh filename=package://robot_properties_fingers/meshes/stl/pro/SIM__BL-F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 scale=1.0 1.0 1.0; visual mesh filename=package://robot_properties_fingers/meshes/stl/pro/SIM__BL-F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 scale=1.0 1.0 1.0
- link finger_tip_link_120: mass 0 -> 0.031; geometry collision mesh filename=package://robot_properties_fingers/meshes/stl/pro/SIM__BL-F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 scale=1.0 1.0 1.0; visual mesh filename=package://robot_properties_fingers/meshes/stl/pro/SIM__BL-F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 scale=1.0 1.0 1.0
- link finger_tip_link_240: mass 0 -> 0.031; geometry collision mesh filename=package://robot_properties_fingers/meshes/stl/pro/SIM__BL-F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 scale=1.0 1.0 1.0; visual mesh filename=package://robot_properties_fingers/meshes/stl/pro/SIM__BL-F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 scale=1.0 1.0 1.0
- link finger_upper_link_0: mass 0.2 -> 0.26
- link finger_upper_link_120: mass 0.2 -> 0.26
- link finger_upper_link_240: mass 0.2 -> 0.26

Commit message: Update robot model
Update robot models to state of robot_properties_fingers rev. c54301e

File: python/trifinger_simulation/robot_properties_fingers/urdf/pro/fingerpro.urdf (robot description, URDF)
Before this commit: robot fingerpro, 6 links, 5 joints
Joints:
- joint finger_base_to_upper_joint: limit lower=-0.9 upper=1.4 effort=1000 velocity=1000 -> lower=-0.33 upper=1.0 effort=1000 velocity=1000
- joint finger_upper_to_middle_joint: limit lower=-1.57 upper=1.57 effort=1000 velocity=1000 -> lower=0.0 upper=1.57 effort=1000 velocity=1000

File: python/trifinger_simulation/robot_properties_fingers/urdf/pro/trifingerpro.urdf (robot description, URDF)
Before this commit: robot trifingerpro, 17 links, 16 joints
Joints:
- joint finger_base_to_upper_joint_0: limit lower=-0.9 upper=1.4 effort=1000 velocity=1000 -> lower=-0.33 upper=1.0 effort=1000 velocity=1000
- joint finger_base_to_upper_joint_120: limit lower=-0.9 upper=1.4 effort=1000 velocity=1000 -> lower=-0.33 upper=1.0 effort=1000 velocity=1000
- joint finger_base_to_upper_joint_240: limit lower=-0.9 upper=1.4 effort=1000 velocity=1000 -> lower=-0.33 upper=1.0 effort=1000 velocity=1000
- joint finger_upper_to_middle_joint_0: limit lower=-1.57 upper=1.57 effort=1000 velocity=1000 -> lower=0.0 upper=1.57 effort=1000 velocity=1000
- joint finger_upper_to_middle_joint_120: limit lower=-1.57 upper=1.57 effort=1000 velocity=1000 -> lower=0.0 upper=1.57 effort=1000 velocity=1000
- joint finger_upper_to_middle_joint_240: limit lower=-1.57 upper=1.57 effort=1000 velocity=1000 -> lower=0.0 upper=1.57 effort=1000 velocity=1000

File: python/trifinger_simulation/robot_properties_fingers/urdf/pro/trifingerpro_with_stage.urdf (robot description, URDF)
Before this commit: robot trifingerpro_with_stage, 19 links, 18 joints
Joints:
- joint finger_base_to_upper_joint_0: limit lower=-0.9 upper=1.4 effort=1000 velocity=1000 -> lower=-0.33 upper=1.0 effort=1000 velocity=1000
- joint finger_base_to_upper_joint_120: limit lower=-0.9 upper=1.4 effort=1000 velocity=1000 -> lower=-0.33 upper=1.0 effort=1000 velocity=1000
- joint finger_base_to_upper_joint_240: limit lower=-0.9 upper=1.4 effort=1000 velocity=1000 -> lower=-0.33 upper=1.0 effort=1000 velocity=1000
- joint finger_upper_to_middle_joint_0: limit lower=-1.57 upper=1.57 effort=1000 velocity=1000 -> lower=0.0 upper=1.57 effort=1000 velocity=1000
- joint finger_upper_to_middle_joint_120: limit lower=-1.57 upper=1.57 effort=1000 velocity=1000 -> lower=0.0 upper=1.57 effort=1000 velocity=1000
- joint finger_upper_to_middle_joint_240: limit lower=-1.57 upper=1.57 effort=1000 velocity=1000 -> lower=0.0 upper=1.57 effort=1000 velocity=1000
