Commit message: Update local copy of robot_properties_fingers

File: python/trifinger_simulation/robot_properties_fingers/urdf/pro/fingerpro.urdf (robot description, URDF)
Before this commit: robot fingerpro, 8 links, 7 joints
Links:
- removed link finger_middle_link_motor
- removed link finger_upper_link_motor
- added link finger_middle_link_visuals, mass 0; visual cylinder length=0.002 radius=0.014; visual cylinder length=0.015 radius=0.005
- added link finger_upper_link_visuals, mass 0; visual cylinder length=0.002 radius=0.014; visual cylinder length=0.015 radius=0.005
- link center_link: geometry collision mesh filename=package://robot_properties_fingers/meshes/pro/center_axis_s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 scale=1.0 1.0 1.0; visual mesh filename=package://robot_properties_fingers/meshes/pro/center_axis_s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 scale=1.0 1.0 1.0
- link finger_base_link: mass 1 -> 0; geometry 
- link finger_lower_link: mass 0.021 -> 0.05569; geometry collision mesh filename=package://robot_properties_fingers/meshes/pro/tip_link_sim.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 scale=1.0 1.0 1.0; visual mesh filename=package://robot_properties_fingers/meshes/pro/tip_link_sim.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 scale=1.0 1.0 1.0
- link finger_middle_link: mass 0.25 -> 0.27163; geometry collision mesh filename=package://robot_properties_fingers/meshes/pro/int_sim.stl scale=1.0 1.0 1.0; visual mesh filename=package://robot_properties_fingers/meshes/pro/int_sim.stl scale=1.0 1.0 1.0
- link finger_tip_link: geometry collision mesh filename=package://robot_properties_fingers/meshes/pro/tip_sim.stl scale=1.0 1.0 1.0; visual mesh filename=package://robot_properties_fingers/meshes/pro/tip_sim.stl scale=1.0 1.0 1.0
- link finger_upper_link: mass 0.26 -> 0.26689; geometry collision mesh filename=package://robot_properties_fingers/meshes/pro/prox-sim.stl scale=1.0 1.0 1.0; visual mesh filename=package://robot_properties_fingers/meshes/pro/prox-sim.stl scale=1.0 1.0 1.0
Joints:
- removed joint finger_middle_to_motor_joint
- removed joint finger_upper_to_motor_joint
- added joint finger_middle_visuals_joint: type fixed, parent finger_middle_link, child finger_middle_link_visuals
- added joint finger_upper_visuals_joint: type fixed, parent finger_upper_link, child finger_upper_link_visuals, origin xyz=0 0 0
- joint finger_lower_to_tip_joint: origin xyz=0.0185 0 -0.1626 -> xyz=0.019 0 -0.16
- joint finger_middle_to_lower_joint: origin xyz=0.04922 0 -0.16 rpy=0 0 0 -> xyz=0.05015 0 -0.16 rpy=0 0 0

File: python/trifinger_simulation/robot_properties_fingers/urdf/pro/trifingerpro.urdf (robot description, URDF)
Before this commit: robot trifingerpro, 23 links, 22 joints
Links:
- removed link finger_middle_link_motor_0
- removed link finger_middle_link_motor_120
- removed link finger_middle_link_motor_240
- removed link finger_upper_link_motor_0
- removed link finger_upper_link_motor_120
- removed link finger_upper_link_motor_240
- added link finger_middle_link_visuals_0, mass 0; visual cylinder length=0.002 radius=0.014; visual cylinder length=0.015 radius=0.005
- added link finger_middle_link_visuals_120, mass 0; visual cylinder length=0.002 radius=0.014; visual cylinder length=0.015 radius=0.005
- added link finger_middle_link_visuals_240, mass 0; visual cylinder length=0.002 radius=0.014; visual cylinder length=0.015 radius=0.005
- added link finger_upper_link_visuals_0, mass 0; visual cylinder length=0.002 radius=0.014; visual cylinder length=0.015 radius=0.005
- added link finger_upper_link_visuals_120, mass 0; visual cylinder length=0.002 radius=0.014; visual cylinder length=0.015 radius=0.005
- added link finger_upper_link_visuals_240, mass 0; visual cylinder length=0.002 radius=0.014; visual cylinder length=0.015 radius=0.005
- link finger_base_link_0: mass 1 -> 0; geometry 
- link finger_base_link_120: mass 1 -> 0; geometry 
- link finger_base_link_240: mass 1 -> 0; geometry 
- link finger_lower_link_0: mass 0.021 -> 0.05569; geometry collision mesh filename=package://robot_properties_fingers/meshes/pro/tip_link_sim.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 scale=1.0 1.0 1.0; visual mesh filename=package://robot_properties_fingers/meshes/pro/tip_link_sim.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 scale=1.0 1.0 1.0
- link finger_lower_link_120: mass 0.021 -> 0.05569; geometry collision mesh filename=package://robot_properties_fingers/meshes/pro/tip_link_sim.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 scale=1.0 1.0 1.0; visual mesh filename=package://robot_properties_fingers/meshes/pro/tip_link_sim.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 scale=1.0 1.0 1.0
- link finger_lower_link_240: mass 0.021 -> 0.05569; geometry collision mesh filename=package://robot_properties_fingers/meshes/pro/tip_link_sim.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 scale=1.0 1.0 1.0; visual mesh filename=package://robot_properties_fingers/meshes/pro/tip_link_sim.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 scale=1.0 1.0 1.0
- link finger_middle_link_0: mass 0.25 -> 0.27163; geometry collision mesh filename=package://robot_properties_fingers/meshes/pro/int_sim.stl scale=1.0 1.0 1.0; visual mesh filename=package://robot_properties_fingers/meshes/pro/int_sim.stl scale=1.0 1.0 1.0
- link finger_middle_link_120: mass 0.25 -> 0.27163; geometry collision mesh filename=package://robot_properties_fingers/meshes/pro/int_sim.stl scale=1.0 1.0 1.0; visual mesh filename=package://robot_properties_fingers/meshes/pro/int_sim.stl scale=1.0 1.0 1.0
- link finger_middle_link_240: mass 0.25 -> 0.27163; geometry collision mesh filename=package://robot_properties_fingers/meshes/pro/int_sim.stl scale=1.0 1.0 1.0; visual mesh filename=package://robot_properties_fingers/meshes/pro/int_sim.stl scale=1.0 1.0 1.0
- link finger_tip_link_0: geometry collision mesh filename=package://robot_properties_fingers/meshes/pro/tip_sim.stl scale=1.0 1.0 1.0; visual mesh filename=package://robot_properties_fingers/meshes/pro/tip_sim.stl scale=1.0 1.0 1.0
- link finger_tip_link_120: geometry collision mesh filename=package://robot_properties_fingers/meshes/pro/tip_sim.stl scale=1.0 1.0 1.0; visual mesh filename=package://robot_properties_fingers/meshes/pro/tip_sim.stl scale=1.0 1.0 1.0
- link finger_tip_link_240: geometry collision mesh filename=package://robot_properties_fingers/meshes/pro/tip_sim.stl scale=1.0 1.0 1.0; visual mesh filename=package://robot_properties_fingers/meshes/pro/tip_sim.stl scale=1.0 1.0 1.0
- link finger_upper_link_0: mass 0.26 -> 0.26689; geometry collision mesh filename=package://robot_properties_fingers/meshes/pro/prox-sim.stl scale=1.0 1.0 1.0; visual mesh filename=package://robot_properties_fingers/meshes/pro/prox-sim.stl scale=1.0 1.0 1.0
- link finger_upper_link_120: mass 0.26 -> 0.26689; geometry collision mesh filename=package://robot_properties_fingers/meshes/pro/prox-sim.stl scale=1.0 1.0 1.0; visual mesh filename=package://robot_properties_fingers/meshes/pro/prox-sim.stl scale=1.0 1.0 1.0
- link finger_upper_link_240: mass 0.26 -> 0.26689; geometry collision mesh filename=package://robot_properties_fingers/meshes/pro/prox-sim.stl scale=1.0 1.0 1.0; visual mesh filename=package://robot_properties_fingers/meshes/pro/prox-sim.stl scale=1.0 1.0 1.0
- link upper_holder_link: mass 1 -> 0; geometry visual mesh filename=package://robot_properties_fingers/meshes/pro/center_axis_s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 scale=1.0 1.0 1.0
Joints:
- removed joint finger_middle_to_motor_joint_0
- removed joint finger_middle_to_motor_joint_120
- removed joint finger_middle_to_motor_joint_240
- removed joint finger_upper_to_motor_joint_0
- removed joint finger_upper_to_motor_joint_120
- removed joint finger_upper_to_motor_joint_240
- added joint finger_middle_visuals_joint_0: type fixed, parent finger_middle_link_0, child finger_middle_link_visuals_0
- added joint finger_middle_visuals_joint_120: type fixed, parent finger_middle_link_120, child finger_middle_link_visuals_120
- added joint finger_middle_visuals_joint_240: type fixed, parent finger_middle_link_240, child finger_middle_link_visuals_240
- added joint finger_upper_visuals_joint_0: type fixed, parent finger_upper_link_0, child finger_upper_link_visuals_0, origin xyz=0 0 0
- added joint finger_upper_visuals_joint_120: type fixed, parent finger_upper_link_120, child finger_upper_link_visuals_120, origin xyz=0 0 0
- added joint finger_upper_visuals_joint_240: type fixed, parent finger_upper_link_240, child finger_upper_link_visuals_240, origin xyz=0 0 0
- joint finger_lower_to_tip_joint_0: origin xyz=0.0185 0 -0.1626 -> xyz=0.019 0 -0.16
- joint finger_lower_to_tip_joint_120: origin xyz=0.0185 0 -0.1626 -> xyz=0.019 0 -0.16
- joint finger_lower_to_tip_joint_240: origin xyz=0.0185 0 -0.1626 -> xyz=0.019 0 -0.16
- joint finger_middle_to_lower_joint_0: origin xyz=0.04922 0 -0.16 rpy=0 0 0 -> xyz=0.05015 0 -0.16 rpy=0 0 0
- joint finger_middle_to_lower_joint_120: origin xyz=0.04922 0 -0.16 rpy=0 0 0 -> xyz=0.05015 0 -0.16 rpy=0 0 0
- joint finger_middle_to_lower_joint_240: origin xyz=0.04922 0 -0.16 rpy=0 0 0 -> xyz=0.05015 0 -0.16 rpy=0 0 0

File: python/trifinger_simulation/robot_properties_fingers/urdf/pro/trifingerpro_with_stage.urdf (robot description, URDF)
Before this commit: robot trifingerpro_with_stage, 25 links, 24 joints
Links:
- removed link finger_middle_link_motor_0
- removed link finger_middle_link_motor_120
- removed link finger_middle_link_motor_240
- removed link finger_upper_link_motor_0
- removed link finger_upper_link_motor_120
- removed link finger_upper_link_motor_240
- added link finger_middle_link_visuals_0, mass 0; visual cylinder length=0.002 radius=0.014; visual cylinder length=0.015 radius=0.005
- added link finger_middle_link_visuals_120, mass 0; visual cylinder length=0.002 radius=0.014; visual cylinder length=0.015 radius=0.005
- added link finger_middle_link_visuals_240, mass 0; visual cylinder length=0.002 radius=0.014; visual cylinder length=0.015 radius=0.005
- added link finger_upper_link_visuals_0, mass 0; visual cylinder length=0.002 radius=0.014; visual cylinder length=0.015 radius=0.005
- added link finger_upper_link_visuals_120, mass 0; visual cylinder length=0.002 radius=0.014; visual cylinder length=0.015 radius=0.005
- added link finger_upper_link_visuals_240, mass 0; visual cylinder length=0.002 radius=0.014; visual cylinder length=0.015 radius=0.005
- link finger_base_link_0: mass 1 -> 0; geometry 
- link finger_base_link_120: mass 1 -> 0; geometry 
- link finger_base_link_240: mass 1 -> 0; geometry 
- link finger_lower_link_0: mass 0.021 -> 0.05569; geometry collision mesh filename=package://robot_properties_fingers/meshes/pro/tip_link_sim.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 scale=1.0 1.0 1.0; visual mesh filename=package://robot_properties_fingers/meshes/pro/tip_link_sim.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 scale=1.0 1.0 1.0
- link finger_lower_link_120: mass 0.021 -> 0.05569; geometry collision mesh filename=package://robot_properties_fingers/meshes/pro/tip_link_sim.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 scale=1.0 1.0 1.0; visual mesh filename=package://robot_properties_fingers/meshes/pro/tip_link_sim.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 scale=1.0 1.0 1.0
- link finger_lower_link_240: mass 0.021 -> 0.05569; geometry collision mesh filename=package://robot_properties_fingers/meshes/pro/tip_link_sim.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 scale=1.0 1.0 1.0; visual mesh filename=package://robot_properties_fingers/meshes/pro/tip_link_sim.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 scale=1.0 1.0 1.0
- link finger_middle_link_0: mass 0.25 -> 0.27163; geometry collision mesh filename=package://robot_properties_fingers/meshes/pro/int_sim.stl scale=1.0 1.0 1.0; visual mesh filename=package://robot_properties_fingers/meshes/pro/int_sim.stl scale=1.0 1.0 1.0
- link finger_middle_link_120: mass 0.25 -> 0.27163; geometry collision mesh filename=package://robot_properties_fingers/meshes/pro/int_sim.stl scale=1.0 1.0 1.0; visual mesh filename=package://robot_properties_fingers/meshes/pro/int_sim.stl scale=1.0 1.0 1.0
- link finger_middle_link_240: mass 0.25 -> 0.27163; geometry collision mesh filename=package://robot_properties_fingers/meshes/pro/int_sim.stl scale=1.0 1.0 1.0; visual mesh filename=package://robot_properties_fingers/meshes/pro/int_sim.stl scale=1.0 1.0 1.0
- link finger_tip_link_0: geometry collision mesh filename=package://robot_properties_fingers/meshes/pro/tip_sim.stl scale=1.0 1.0 1.0; visual mesh filename=package://robot_properties_fingers/meshes/pro/tip_sim.stl scale=1.0 1.0 1.0
- link finger_tip_link_120: geometry collision mesh filename=package://robot_properties_fingers/meshes/pro/tip_sim.stl scale=1.0 1.0 1.0; visual mesh filename=package://robot_properties_fingers/meshes/pro/tip_sim.stl scale=1.0 1.0 1.0
- link finger_tip_link_240: geometry collision mesh filename=package://robot_properties_fingers/meshes/pro/tip_sim.stl scale=1.0 1.0 1.0; visual mesh filename=package://robot_properties_fingers/meshes/pro/tip_sim.stl scale=1.0 1.0 1.0
- link finger_upper_link_0: mass 0.26 -> 0.26689; geometry collision mesh filename=package://robot_properties_fingers/meshes/pro/prox-sim.stl scale=1.0 1.0 1.0; visual mesh filename=package://robot_properties_fingers/meshes/pro/prox-sim.stl scale=1.0 1.0 1.0
- link finger_upper_link_120: mass 0.26 -> 0.26689; geometry collision mesh filename=package://robot_properties_fingers/meshes/pro/prox-sim.stl scale=1.0 1.0 1.0; visual mesh filename=package://robot_properties_fingers/meshes/pro/prox-sim.stl scale=1.0 1.0 1.0
- link finger_upper_link_240: mass 0.26 -> 0.26689; geometry collision mesh filename=package://robot_properties_fingers/meshes/pro/prox-sim.stl scale=1.0 1.0 1.0; visual mesh filename=package://robot_properties_fingers/meshes/pro/prox-sim.stl scale=1.0 1.0 1.0
- link upper_holder_link: mass 1 -> 0; geometry visual mesh filename=package://robot_properties_fingers/meshes/pro/center_axis_s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 scale=1.0 1.0 1.0
Joints:
- removed joint finger_middle_to_motor_joint_0
- removed joint finger_middle_to_motor_joint_120
- removed joint finger_middle_to_motor_joint_240
- removed joint finger_upper_to_motor_joint_0
- removed joint finger_upper_to_motor_joint_120
- removed joint finger_upper_to_motor_joint_240
- added joint finger_middle_visuals_joint_0: type fixed, parent finger_middle_link_0, child finger_middle_link_visuals_0
- added joint finger_middle_visuals_joint_120: type fixed, parent finger_middle_link_120, child finger_middle_link_visuals_120
- added joint finger_middle_visuals_joint_240: type fixed, parent finger_middle_link_240, child finger_middle_link_visuals_240
- added joint finger_upper_visuals_joint_0: type fixed, parent finger_upper_link_0, child finger_upper_link_visuals_0, origin xyz=0 0 0
- added joint finger_upper_visuals_joint_120: type fixed, parent finger_upper_link_120, child finger_upper_link_visuals_120, origin xyz=0 0 0
- added joint finger_upper_visuals_joint_240: type fixed, parent finger_upper_link_240, child finger_upper_link_visuals_240, origin xyz=0 0 0
- joint finger_lower_to_tip_joint_0: origin xyz=0.0185 0 -0.1626 -> xyz=0.019 0 -0.16
- joint finger_lower_to_tip_joint_120: origin xyz=0.0185 0 -0.1626 -> xyz=0.019 0 -0.16
- joint finger_lower_to_tip_joint_240: origin xyz=0.0185 0 -0.1626 -> xyz=0.019 0 -0.16
- joint finger_middle_to_lower_joint_0: origin xyz=0.04922 0 -0.16 rpy=0 0 0 -> xyz=0.05015 0 -0.16 rpy=0 0 0
- joint finger_middle_to_lower_joint_120: origin xyz=0.04922 0 -0.16 rpy=0 0 0 -> xyz=0.05015 0 -0.16 rpy=0 0 0
- joint finger_middle_to_lower_joint_240: origin xyz=0.04922 0 -0.16 rpy=0 0 0 -> xyz=0.05015 0 -0.16 rpy=0 0 0

File: python/trifinger_simulation/robot_properties_fingers/urdf/trifinger.urdf (robot description, URDF)
Before this commit: robot finger_with_stage, 17 links, 16 joints
Joints:
- joint base_to_upper_holder_joint: origin xyz=0 0 0.34 -> xyz=0 0 0.29

File: python/trifinger_simulation/robot_properties_fingers/urdf/trifinger_with_stage.urdf (robot description, URDF)
Before this commit: robot trifinger_with_stage, 19 links, 18 joints
Joints:
- joint base_to_upper_holder_joint: origin xyz=0 0 0.34 -> xyz=0 0 0.29

Commit message: Update copy of robot_properties_fingers
Update the local copy of the robot model to the state of
robot_properties_fingers git revision 1257ff7.

File: python/trifinger_simulation/robot_properties_fingers/urdf/pro/fingerpro.urdf (robot description, URDF)
Before this commit: robot fingerpro, 8 links, 7 joints
Links:
- added link base_link, mass 0
Joints:
- added joint base_to_center_joint: type fixed, parent base_link, child center_link, origin xyz=0 0 0.29

File: python/trifinger_simulation/robot_properties_fingers/urdf/pro/trifingerpro.urdf (robot description, URDF)
Before this commit: robot trifingerpro, 23 links, 22 joints
Links:
- link base_link: mass 1 -> 0

File: python/trifinger_simulation/robot_properties_fingers/urdf/pro/trifingerpro_with_stage.urdf (robot description, URDF)
Before this commit: robot trifingerpro_with_stage, 25 links, 24 joints
Links:
- link base_link: mass 1 -> 0
