Commit message: fix: Update URDF files with latest version from robot_properties_fingers
Taken from robot_properties_fingers commit
427200b22ee4e595cf9a3b67d935698a44eb8ef2.

File: trifinger_simulation/robot_properties_fingers/urdf/pro/fingerpro.urdf (robot description, URDF)
Before this commit: robot fingerpro, 9 links, 8 joints
Links:
- link finger_tip_link: mass 0.031 -> 0.0092

File: trifinger_simulation/robot_properties_fingers/urdf/pro/trifingerpro.urdf (robot description, URDF)
Before this commit: robot trifingerpro, 23 links, 22 joints
Links:
- link finger_tip_link_0: mass 0.031 -> 0.0092
- link finger_tip_link_120: mass 0.031 -> 0.0092
- link finger_tip_link_240: mass 0.031 -> 0.0092

File: trifinger_simulation/robot_properties_fingers/urdf/pro/trifingerpro_with_stage.urdf (robot description, URDF)
Before this commit: robot trifingerpro_with_stage, 25 links, 24 joints
Links:
- link finger_tip_link_0: mass 0.031 -> 0.0092
- link finger_tip_link_120: mass 0.031 -> 0.0092
- link finger_tip_link_240: mass 0.031 -> 0.0092
